File: Skis.sch (KiCad schematic (older format))
At the start: 96 parts, among them J1 TRIG_A, J10 SIGNAL_OUT_B, J11 ENV_OUT_B, J2 CV_IN_A, J3 SIGNAL_IN_A, J4 SIGNAL_OUT_A, J5 ENV_OUT_A, J6 EuroPower, J7 TRIG_B, J8 CV_IN_B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

Commit message: Added normalization for input jacks
Connections:
- net GND: no longer J9.TN
- net NORM_IN: now reaches J3.T, Q1.3 (D), SW1.1 (A)
- net NORM_IN: now also J9.TN
Changed lines of the file:
@@
 Wire Wire Line
 	1350 4200 1450 4200
-Wire Wire Line
-	1450 4200 1450 4400
-Connection ~ 1450 4400
 $Comp
 L Switch:SW_SPDT SW1
@@
 Wire Wire Line
 	9300 4300 9400 4300
-Wire Wire Line
-	9400 4300 9400 4500
-Connection ~ 9400 4500
 $Comp
 L Switch:SW_SPDT SW3
@@
 	1    0    0    -1
 $EndComp
+Text GLabel 9400 4300 2    50   Input ~ 0
+NORM_IN
+Text GLabel 1900 4200 1    50   Input ~ 0
+NORM_IN
+Connection ~ 1450 4400
+Wire Wire Line
+	1450 4200 1450 4400
+Wire Wire Line
+	1900 4200 1900 4300
 $EndSCHEMATC
